File: Data_acquisition_circuit/AQ.kicad_sch (KiCad schematic)
At the start: 0 parts

Commit message: add amplifier, adc and rewrite power file
Parts:
- added U14: AD8630ARZ, R_14_ADI, symbol AD8630ARZ:AD8630ARZ
Changed lines of the file:
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@@
 (kicad_sch (version 20230121) (generator eeschema)
   (paper "A4")
+  (symbol (lib_id "AD8630ARZ:AD8630ARZ") (at 109.22 64.77 0) (unit 1)
+    (in_bom yes) (on_board yes) (dnp no) (fields_autoplaced)
+    (property "Reference" "U14" (at 139.7 54.61 0)
+      (effects (font (size 1.524 1.524)))
+    )
+    (property "Value" "AD8630ARZ" (at 139.7 57.15 0)
+      (effects (font (size 1.524 1.524)))
+    )
+    (property "Footprint" "R_14_ADI" (at 109.22 64.77 0)
+      (effects (font (size 1.27 1.27) italic) hide)
+    )
+    (property "Datasheet" "AD8630ARZ" (at 109.22 64.77 0)
+      (effects (font (size 1.27 1.27) italic) hide)
+    )
+    (pin "1")
+    (pin "10")
+    (pin "11")
+    (pin "12")
+    (pin "13")
+    (pin "14")
+    (pin "2")
+    (pin "3")
+    (pin "4")
+    (pin "5")
+    (pin "6")
+    (pin "7")
+    (pin "8")
+    (pin "9")
+    (instances
+      (project "Data acquisition circuit"
+        (path "/1b7d87d8-ce09-4d95-b010-1b82030051eb/64241bff-6be2-4de8-ab96-8d24081a216d"
+          (reference "U14") (unit 1)
+        )
+        (path "/1b7d87d8-ce09-4d95-b010-1b82030051eb/fc24ae42-38bb-47e7-b5cf-739ccf1d1089"
+          (reference "U14") (unit 1)
+        )
+      )
+    )
+  )
 )
